File: kicad/Keyboard.kicad_pcb (KiCad board)
At the start: 2 copper layers, 3.6 x 3.3 mm, 124 parts, among them J1 Conn_01x03_Pin, J10 Conn_01x03_Pin, J11 Conn_01x04_Pin, J12 Conn_01x03_Pin, J2 AudioJack4, J3 AudioJack4, J4 Conn_01x04_Pin, J5 Conn_01x04_Pin, J6 Conn_01x04_Pin, J7 Conn_01x03_Pin, J8 Conn_01x03_Pin, J9 Conn_01x04_Pin, SW1 SW_Push, SW10 SW_Push, SW11 SW_Push, SW12 SW_Push, SW13 SW_Push, SW14 SW_Push, SW15 SW_Push, SW16 SW_Push, SW17 SW_Push, SW18 SW_Push, SW19 SW_Push, SW2 SW_Push, SW20 SW_Push, SW21 SW_Push, SW22 SW_Push, SW23 SW_Push, SW24 SW_Push, SW25 SW_Push, SW26 SW_Push, SW27 SW_Push, SW28 SW_Push, SW29 SW_Push, SW3 SW_Push, SW30 SW_Push, SW31 SW_Push, SW32 SW_Push, SW33 SW_Push, SW34 SW_Push, SW35 SW_Push, SW36 SW_Push, SW4 SW_Push, SW5 SW_Push, SW6 SW_Push, SW7 SW_Push, SW8 SW_Push, SW9 SW_Push, U1 RP2040-Zero, U2 RP2040-Zero

Commit message: wip: pcb for both halves
Parts:
- SW1, SW10, SW11, SW12, SW13, SW14, SW15, SW16, SW17, SW18, SW19, SW2, SW20, SW21, SW22, SW23, SW24, SW25, SW26, SW27, SW28, SW29, SW3, SW30, SW31, SW32, SW33, SW34, SW35, SW36, SW4, SW5, SW6, SW7, SW8, SW9: footprint Choc-V1:SW_Kailh_Choc_V1 -> Choc-V1:SW_Kailh_Choc_V1_THT
- moved J1 260.7 mm to (-77.4, 34.8), turned to -90 degrees
- moved U1 250.3 mm to (-71.9, 46.8)
- moved J7 246.6 mm to (-86.9, 70.5), turned to 180 degrees
- moved R2 238.9 mm to (-74.4, 35.9), turned to 90 degrees
- moved R1 237.8 mm to (-79.9, 31.7), turned to 90 degrees
- moved J2 237.7 mm to (-57.6, 35.7), turned to 180 degrees
- moved J6 237.6 mm to (-79.8, 61.9), turned to -90 degrees
- moved D16 236.9 mm to (-81.8, 80.6), turned to -15 degrees
- moved D49 220.4 mm to (-68.8, 73.9), turned to 165 degrees
- moved D17 219.6 mm to (-64.4, 85.9), turned to -30 degrees
- moved SW16 212.8 mm to (-72.4, 73.3), turned to -15 degrees
- moved D72 211.0 mm to (120.3, 103.9), turned to 45 degrees
- moved D18 203.6 mm to (-49.3, 94.9), turned to -45 degrees
- moved J8 202.9 mm to (-90.4, 65.5)
- moved D50 201.6 mm to (-49.9, 82.8), turned to 150 degrees
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Connections:
- D1 pad 1: (no net) -> /Left Half/R1
- D1 pad 2: (no net) -> Net-(D1-A)
- D10 pad 1: /Left Half/C1 -> /Left Half/R2
- D10 pad 2: (no net) -> Net-(D10-A)
- D11 pad 1: /Left Half/C1 -> /Left Half/R3
- D11 pad 2: (no net) -> Net-(D11-A)
- D12 pad 1: /Left Half/C1 -> /Left Half/R3
- D12 pad 2: (no net) -> Net-(D12-A)
- D13 pad 1: /Left Half/C1 -> /Left Half/R3
- D13 pad 2: (no net) -> Net-(D13-A)
- D14 pad 1: /Left Half/C1 -> /Left Half/R3
- D14 pad 2: (no net) -> Net-(D14-A)
- D15 pad 1: /Left Half/C1 -> /Left Half/R3
- D15 pad 2: (no net) -> Net-(D15-A)
- D16 pad 1: (no net) -> /Left Half/Thumbpad/R1
- D16 pad 2: (no net) -> Net-(D16-A)
- D17 pad 1: Net-(D16-K) -> /Left Half/Thumbpad/R2
- D17 pad 2: (no net) -> Net-(D17-A)
- D18 pad 1: Net-(D16-K) -> /Left Half/Thumbpad/R3
- D18 pad 2: (no net) -> Net-(D18-A)
- D19 pad 1: (no net) -> /Right Half/R1
- D19 pad 2: (no net) -> Net-(D19-A)
- D2 pad 1: /Left Half/C1 -> /Left Half/R1
- D2 pad 2: (no net) -> Net-(D2-A)
- D20 pad 1: /Right Half/C1 -> /Right Half/R2
- D20 pad 2: (no net) -> Net-(D20-A)
- D21 pad 1: /Right Half/C1 -> /Right Half/R3
- D21 pad 2: (no net) -> Net-(D21-A)
- D22 pad 1: /Right Half/C1 -> /Right Half/R1
- D22 pad 2: (no net) -> Net-(D22-A)
- D23 pad 1: /Right Half/C1 -> /Right Half/R2
- D23 pad 2: (no net) -> Net-(D23-A)
- D24 pad 1: /Right Half/C1 -> /Right Half/R3
- D24 pad 2: (no net) -> Net-(D24-A)
- D25 pad 1: /Right Half/C1 -> /Right Half/R1
- D25 pad 2: (no net) -> Net-(D25-A)
- D26 pad 1: /Right Half/C1 -> /Right Half/R2
- D26 pad 2: (no net) -> Net-(D26-A)
- D27 pad 1: /Right Half/C1 -> /Right Half/R3
- D27 pad 2: (no net) -> Net-(D27-A)
- D28 pad 1: (no net) -> Net-(D28-DOUT)
- D28 pad 2: (no net) -> GND
- D28 pad 3: (no net) -> Net-(D28-DIN)
- D28 pad 4: (no net) -> +5V
- D29 pad 2: /Right Half/GND -> GND
- D29 pad 3: (no net) -> Net-(D29-DIN)
- D29 pad 4: /Right Half/VCC_5V -> +5V
- D3 pad 1: /Left Half/C1 -> /Left Half/R1
- D3 pad 2: (no net) -> Net-(D3-A)
- D30 pad 1: (no net) -> Net-(D30-DOUT)
- D30 pad 2: /Right Half/GND -> GND
- D30 pad 3: (no net) -> Net-(D30-DIN)
- D30 pad 4: /Right Half/VCC_5V -> +5V
- D31 pad 1: (no net) -> Net-(D31-DOUT)
- D31 pad 2: /Right Half/GND -> GND
- D31 pad 4: /Right Half/VCC_5V -> +5V
- D32 pad 2: /Right Half/GND -> GND
- D32 pad 3: (no net) -> Net-(D32-DIN)
- D32 pad 4: /Right Half/VCC_5V -> +5V
- D33 pad 2: /Right Half/GND -> GND
- D33 pad 3: (no net) -> Net-(D33-DIN)
- D33 pad 4: /Right Half/VCC_5V -> +5V
- D34 pad 1: /Right Half/C1 -> /Right Half/R1
- D34 pad 2: (no net) -> Net-(D34-A)
- D35 pad 1: /Right Half/C1 -> /Right Half/R2
- D35 pad 2: (no net) -> Net-(D35-A)
- D36 pad 1: /Right Half/C1 -> /Right Half/R3
- D36 pad 2: (no net) -> Net-(D36-A)
- D37 pad 1: (no net) -> Net-(D37-DOUT)
- D37 pad 2: (no net) -> GND
- D37 pad 3: (no net) -> /Left Half/DIN
- D37 pad 4: (no net) -> +5V
- D38 pad 1: (no net) -> Net-(D38-DOUT)
- D38 pad 2: /Left Half/GND -> GND
- D38 pad 4: /Left Half/VCC_5V -> +5V
- D39 pad 1: (no net) -> Net-(D39-DOUT)
- D39 pad 2: /Left Half/GND -> GND
- D39 pad 4: /Left Half/VCC_5V -> +5V
- D4 pad 1: /Left Half/C1 -> /Left Half/R1
- D4 pad 2: (no net) -> Net-(D4-A)
- D40 pad 1: (no net) -> Net-(D40-DOUT)
- D40 pad 2: /Left Half/GND -> GND
- D40 pad 4: /Left Half/VCC_5V -> +5V
- D41 pad 1: (no net) -> Net-(D41-DOUT)
- D41 pad 2: /Left Half/GND -> GND
- D41 pad 4: /Left Half/VCC_5V -> +5V
- D42 pad 1: (no net) -> Net-(D42-DOUT)
- D42 pad 2: /Left Half/GND -> GND
- D42 pad 4: /Left Half/VCC_5V -> +5V
- D43 pad 1: (no net) -> Net-(D43-DOUT)
- D43 pad 2: /Left Half/GND -> GND
- D43 pad 3: (no net) -> Net-(D43-DIN)
- D43 pad 4: /Left Half/VCC_5V -> +5V
- D44 pad 2: /Left Half/GND -> GND
- D44 pad 3: (no net) -> Net-(D44-DIN)
- D44 pad 4: /Left Half/VCC_5V -> +5V
- D45 pad 2: /Left Half/GND -> GND
- D45 pad 3: (no net) -> Net-(D45-DIN)
- D45 pad 4: /Left Half/VCC_5V -> +5V
- D46 pad 2: /Left Half/GND -> GND
- D46 pad 3: (no net) -> Net-(D46-DIN)
- D46 pad 4: /Left Half/VCC_5V -> +5V
- D47 pad 2: /Left Half/GND -> GND
- D47 pad 3: (no net) -> Net-(D47-DIN)
- D47 pad 4: /Left Half/VCC_5V -> +5V
- D48 pad 2: /Left Half/GND -> GND
- D48 pad 4: /Left Half/VCC_5V -> +5V
- D49 pad 1: (no net) -> Net-(D49-DOUT)
- D49 pad 2: (no net) -> Net-(D49-VSS)
- D49 pad 3: (no net) -> Net-(D49-DIN)
- D49 pad 4: (no net) -> Net-(D49-VDD)
- D5 pad 1: /Left Half/C1 -> /Left Half/R1
- D5 pad 2: (no net) -> Net-(D5-A)
- D50 pad 1: (no net) -> Net-(D50-DOUT)
- D51 pad 1: (no net) -> unconnected-(D51-DOUT-Pad1)
- D52 pad 1: (no net) -> Net-(D52-DOUT)
- D52 pad 2: /Left Half/GND -> GND
- D52 pad 3: (no net) -> Net-(D52-DIN)
- D52 pad 4: /Left Half/VCC_5V -> +5V
- D53 pad 2: /Left Half/GND -> GND
- D53 pad 3: (no net) -> Net-(D53-DIN)
- D53 pad 4: /Left Half/VCC_5V -> +5V
- D54 pad 2: /Left Half/GND -> GND
- D54 pad 4: /Left Half/VCC_5V -> +5V
- D55 pad 1: (no net) -> Net-(D55-DOUT)
- D55 pad 2: /Right Half/GND -> GND
- D55 pad 4: /Right Half/VCC_5V -> +5V
- D56 pad 2: /Right Half/GND -> GND
- D56 pad 3: (no net) -> Net-(D56-DIN)
- D56 pad 4: /Right Half/VCC_5V -> +5V
- D57 pad 2: /Right Half/GND -> GND
- D57 pad 3: (no net) -> Net-(D57-DIN)
- D57 pad 4: /Right Half/VCC_5V -> +5V
- D58 pad 1: /Right Half/C1 -> /Right Half/R1
- D58 pad 2: (no net) -> Net-(D58-A)
- D59 pad 1: /Right Half/C1 -> /Right Half/R2
- D59 pad 2: (no net) -> Net-(D59-A)
- D6 pad 1: /Left Half/C1 -> /Left Half/R2
- D6 pad 2: (no net) -> Net-(D6-A)
- D60 pad 1: /Right Half/C1 -> /Right Half/R3
- D60 pad 2: (no net) -> Net-(D60-A)
- D61 pad 1: (no net) -> Net-(D61-DOUT)
- D61 pad 2: /Right Half/GND -> GND
- D61 pad 4: /Right Half/VCC_5V -> +5V
- D62 pad 2: /Right Half/GND -> GND
- D62 pad 3: (no net) -> Net-(D62-DIN)
- D62 pad 4: /Right Half/VCC_5V -> +5V
- D63 pad 2: /Right Half/GND -> GND
- D63 pad 3: (no net) -> Net-(D63-DIN)
- D63 pad 4: /Right Half/VCC_5V -> +5V
- D64 pad 1: (no net) -> Net-(D64-DOUT)
- D64 pad 2: /Right Half/GND -> GND
- D64 pad 4: /Right Half/VCC_5V -> +5V
- D65 pad 2: /Right Half/GND -> GND
- D65 pad 4: /Right Half/VCC_5V -> +5V
- D66 pad 2: /Right Half/GND -> GND
- D66 pad 3: (no net) -> /Right Half/DIN
- D66 pad 4: /Right Half/VCC_5V -> +5V
- D67 pad 1: (no net) -> Net-(D67-DOUT)
- D67 pad 2: (no net) -> Net-(D67-VSS)
- D67 pad 3: (no net) -> Net-(D67-DIN)
- D67 pad 4: (no net) -> Net-(D67-VDD)
- D68 pad 1: (no net) -> /Right Half/Thumbpad/R1
- D68 pad 2: (no net) -> Net-(D68-A)
- D69 pad 1: Net-(D68-K) -> /Right Half/Thumbpad/R2
- D69 pad 2: (no net) -> Net-(D69-A)
- D7 pad 1: /Left Half/C1 -> /Left Half/R2
- D7 pad 2: (no net) -> Net-(D7-A)
- D70 pad 1: Net-(D68-K) -> /Right Half/Thumbpad/R3
- D70 pad 2: (no net) -> Net-(D70-A)
- D71 pad 1: (no net) -> Net-(D71-DOUT)
- D72 pad 1: (no net) -> unconnected-(D72-DOUT-Pad1)
- D8 pad 1: /Left Half/C1 -> /Left Half/R2
- D8 pad 2: (no net) -> Net-(D8-A)
- D9 pad 1: /Left Half/C1 -> /Left Half/R2
- D9 pad 2: (no net) -> Net-(D9-A)
- J1 pad 1: /Left Half/GND -> GND
- J1 pad 2: (no net) -> /Left Half/OUT
- J1 pad 3: (no net) -> +5V
- J10 pad 1: /Right Half/GND -> GND
- J10 pad 3: /Right Half/VCC_5V -> +5V
- J11 pad 1: Net-(D68-K) -> /Right Half/Thumbpad/C1
- J11 pad 2: Net-(D68-K) -> /Right Half/Thumbpad/R1
- J11 pad 3: Net-(D68-K) -> /Right Half/Thumbpad/R2
- J11 pad 4: Net-(D68-K) -> /Right Half/Thumbpad/R3
- J2 pad 1: (no net) -> GND
- J2 pad 2: (no net) -> +5V
- J2 pad 3: (no net) -> /Left Half/Tx
- J2 pad 4: (no net) -> /Left Half/Rx
- J3 pad 1: (no net) -> GND
- J3 pad 2: (no net) -> +5V
- J3 pad 3: (no net) -> /Right Half/Rx
- J3 pad 4: (no net) -> /Right Half/Tx
- J4 pad 1: (no net) -> /Right Half/SDA
- J4 pad 2: (no net) -> /Right Half/SCL
- J4 pad 3: /Right Half/GND -> GND
- J4 pad 4: /Right Half/VCC_5V -> +5V
- J5 pad 1: /Left Half/C1 -> /Left Half/R3
- J5 pad 2: /Left Half/C1 -> /Left Half/R2
- J5 pad 3: /Left Half/C1 -> /Left Half/R1
- J5 pad 4: (no net) -> /Left Half/C6
- J6 pad 1: Net-(D16-K) -> /Left Half/Thumbpad/C1
- J6 pad 2: Net-(D16-K) -> /Left Half/Thumbpad/R1
- J6 pad 3: Net-(D16-K) -> /Left Half/Thumbpad/R2
- J6 pad 4: Net-(D16-K) -> /Left Half/Thumbpad/R3
- J8 pad 1: /Left Half/GND -> GND
- J8 pad 3: /Left Half/VCC_5V -> +5V
- J9 pad 1: /Right Half/C1 -> /Right Half/R3
- J9 pad 2: /Right Half/C1 -> /Right Half/R2
- J9 pad 3: /Right Half/C1 -> /Right Half/R1
- J9 pad 4: (no net) -> /Right Half/C6
- R1 pad 1: /Left Half/VCC -> /Left Half/OUT
- R1 pad 2: (no net) -> /Left Half/ADC0
- R2 pad 1: /Left Half/GND -> GND
- SW10 pad 2: /Left Half/C1 -> /Left Half/C5
- SW12 pad 2: /Left Half/C1 -> /Left Half/C2
- SW13 pad 2: /Left Half/C1 -> /Left Half/C3
- SW14 pad 2: /Left Half/C1 -> /Left Half/C4
- SW15 pad 2: /Left Half/C1 -> /Left Half/C5
- SW16 pad 2: Net-(D16-K) -> /Left Half/Thumbpad/C1
- SW17 pad 2: Net-(D16-K) -> /Left Half/Thumbpad/C1
- SW18 pad 2: Net-(D16-K) -> /Left Half/Thumbpad/C1
- SW2 pad 2: /Left Half/C1 -> /Left Half/C2
- SW22 pad 2: /Right Half/C1 -> /Right Half/C2
- SW23 pad 2: /Right Half/C1 -> /Right Half/C2
- SW24 pad 2: /Right Half/C1 -> /Right Half/C2
- SW25 pad 2: /Right Half/C1 -> /Right Half/C3
- SW26 pad 2: /Right Half/C1 -> /Right Half/C3
- SW27 pad 2: /Right Half/C1 -> /Right Half/C3
- SW28 pad 2: /Right Half/C1 -> /Right Half/C4
- SW29 pad 2: /Right Half/C1 -> /Right Half/C4
- SW3 pad 2: /Left Half/C1 -> /Left Half/C3
- SW30 pad 2: /Right Half/C1 -> /Right Half/C4
- SW31 pad 2: /Right Half/C1 -> /Right Half/C5
- SW32 pad 2: /Right Half/C1 -> /Right Half/C5
- SW33 pad 2: /Right Half/C1 -> /Right Half/C5
- SW34 pad 2: Net-(D68-K) -> /Right Half/Thumbpad/C1
- SW35 pad 2: Net-(D68-K) -> /Right Half/Thumbpad/C1
- SW36 pad 2: Net-(D68-K) -> /Right Half/Thumbpad/C1
- SW4 pad 2: /Left Half/C1 -> /Left Half/C4
- SW5 pad 2: /Left Half/C1 -> /Left Half/C5
- SW7 pad 2: /Left Half/C1 -> /Left Half/C2
- SW8 pad 2: /Left Half/C1 -> /Left Half/C3
- SW9 pad 2: /Left Half/C1 -> /Left Half/C4
- U1 pad 0: (no net) -> /Left Half/Tx
- U1 pad 1: (no net) -> /Left Half/Rx
- U1 pad 10: /Left Half/C1 -> /Left Half/C2
- U1 pad 11: /Left Half/C1 -> /Left Half/C3
- U1 pad 12: /Left Half/C1 -> /Left Half/C4
- U1 pad 13: /Left Half/C6 -> /Left Half/C5
- U1 pad 14: (no net) -> unconnected-(U1-Pad14)
- U1 pad 2: (no net) -> unconnected-(U1-Pad2)
- U1 pad 27: (no net) -> unconnected-(U1-Pad27)
- U1 pad 28: /Left Half/OUT -> unconnected-(U1-Pad28)
- U1 pad 29: (no net) -> unconnected-(U1-Pad29)
- U1 pad 3: (no net) -> unconnected-(U1-Pad3)
- U1 pad 3v3: /Left Half/VCC -> unconnected-(U1-Pad3v3)
- U1 pad 4: (no net) -> unconnected-(U1-Pad4)
- U1 pad 5: /Left Half/C1 -> /Left Half/C6
- U1 pad 5v: /Left Half/VCC_5V -> +5V
- U1 pad 6: /Left Half/C1 -> /Left Half/R1
- U1 pad 7: /Left Half/C1 -> /Left Half/R2
- U1 pad 8: /Left Half/C1 -> /Left Half/R3
- U1 pad GND: /Left Half/GND -> GND
- U2 pad 0: (no net) -> /Right Half/Tx
- U2 pad 1: (no net) -> /Right Half/Rx
- U2 pad 10: /Right Half/C1 -> /Right Half/C3
- U2 pad 11: /Right Half/C1 -> /Right Half/C4
- U2 pad 12: /Right Half/C1 -> /Right Half/C5
- U2 pad 13: /Right Half/C6 -> unconnected-(U2-Pad13)
- U2 pad 14: (no net) -> unconnected-(U2-Pad14)
- U2 pad 15: /Right Half/DIN -> /Right Half/C6
- U2 pad 2: (no net) -> unconnected-(U2-Pad2)
- U2 pad 28: (no net) -> unconnected-(U2-Pad28)
- U2 pad 29: (no net) -> unconnected-(U2-Pad29)
- U2 pad 3: (no net) -> unconnected-(U2-Pad3)
- U2 pad 3v3: (no net) -> unconnected-(U2-Pad3v3)
- U2 pad 4: (no net) -> /Right Half/DIN
- U2 pad 5: /Right Half/C1 -> /Right Half/R1
- U2 pad 5v: /Right Half/VCC_5V -> +5V
- U2 pad 6: /Right Half/C1 -> /Right Half/R2
- U2 pad 7: /Right Half/C1 -> /Right Half/R3
- U2 pad 9: /Right Half/C1 -> /Right Half/C2
- U2 pad GND: /Right Half/GND -> GND
Routing:
- net GND: track 0.00 -> 1014.0 mm
- net +5V: track 0.00 -> 962.9 mm
- net (no net): track 270.2 -> 0.00 mm
- net /Left Half/R1: track 0.00 -> 264.8 mm
- net /Left Half/GND: track 230.8 -> 0.00 mm
- net /Right Half/C5: track 0.00 -> 169.1 mm
- net /Right Half/R1: track 0.00 -> 158.4 mm
- net /Right Half/R3: track 0.00 -> 143.2 mm
- net /Left Half/C2: track 0.00 -> 140.3 mm
- net /Left Half/R2: track 0.00 -> 130.8 mm
- net /Right Half/C4: track 0.00 -> 126.6 mm
- net /Right Half/R2: track 0.00 -> 126.1 mm
- net /Left Half/C3: track 0.00 -> 118.7 mm
- net /Left Half/R3: track 0.00 -> 116.4 mm
- net /Right Half/C3: track 0.00 -> 96.9 mm
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Other:
- board size 3.6 x 3.3 mm -> 4.4 x 4.4 mm

Commit message: final PCB ready
- bugs: LED position and wiring (wrong by footprint)
Parts:
- removed J1: Conn_01x03_Pin, Connector_PinHeader_2.54mm:PinHeader_1x03_P2.54mm_Vertical
- removed J4: Conn_01x04_Pin, Connector_PinHeader_2.54mm:PinHeader_1x04_P2.54mm_Vertical
- added REF**: MountingHole_2.2mm_M2, MountingHole:MountingHole_2.2mm_M2, F.Cu at (29.6, 96.0)
- added REF**: MountingHole_2.2mm_M2, MountingHole:MountingHole_2.2mm_M2, F.Cu at (174.0, 104.0)
- added REF**: MountingHole_2.2mm_M2, MountingHole:MountingHole_2.2mm_M2, F.Cu at (274.0, 151.0)
- added REF**: MountingHole_2.2mm_M2, MountingHole:MountingHole_2.2mm_M2, F.Cu at (269.1, 82.7)
- added REF**: MountingHole_2.2mm_M2, MountingHole:MountingHole_2.2mm_M2, F.Cu at (220.0, 110.0)
- added REF**: MountingHole_2.2mm_M2, MountingHole:MountingHole_2.2mm_M2, F.Cu at (86.0, 105.0)
- added REF**: MountingHole_2.2mm_M2, MountingHole:MountingHole_2.2mm_M2, F.Cu at (30.5, 144.8)
- added REF**: MountingHole_2.2mm_M2, MountingHole:MountingHole_2.2mm_M2, F.Cu at (66.0, 56.0)
- added REF**: MountingHole_2.2mm_M2, MountingHole:MountingHole_2.2mm_M2, F.Cu at (23.2, 96.8)
- added REF**: MountingHole_2.2mm_M2, MountingHole:MountingHole_2.2mm_M2, F.Cu at (131.0, 104.0)
- added REF**: MountingHole_2.2mm_M2, MountingHole:MountingHole_2.2mm_M2, F.Cu at (120.0, 136.0)
- added REF**: MountingHole_2.2mm_M2, MountingHole:MountingHole_2.2mm_M2, F.Cu at (207.0, 70.0)
- added REF**: MountingHole_2.2mm_M2, MountingHole:MountingHole_2.2mm_M2, F.Cu at (187.7, 136.2)
- added REF**: MountingHole_2.2mm_M2, MountingHole:MountingHole_2.2mm_M2, F.Cu at (273.8, 97.9)
- added mouse-bite-1mm-3mm: VAL**, Mouse-Bites:mouse-bite-1mm-3mm, F.Cu at (59.0, 77.7)
- added mouse-bite-1mm-3mm: VAL**, Mouse-Bites:mouse-bite-1mm-3mm, F.Cu at (222.2, 77.0)
- added mouse-bite-1mm-3mm: VAL**, Mouse-Bites:mouse-bite-1mm-3mm, F.Cu at (68.2, 70.2)
- added mouse-bite-1mm-3mm: VAL**, Mouse-Bites:mouse-bite-1mm-3mm, F.Cu at (224.3, 79.1)
- added mouse-bite-1mm-3mm: VAL**, Mouse-Bites:mouse-bite-1mm-3mm, F.Cu at (74.2, 70.2)
- added mouse-bite-1mm-3mm: VAL**, Mouse-Bites:mouse-bite-1mm-3mm, F.Cu at (249.6, 92.0)
- added mouse-bite-1mm-3mm: VAL**, Mouse-Bites:mouse-bite-1mm-3mm, F.Cu at (153.3, 113.0)
- added mouse-bite-1mm-3mm: VAL**, Mouse-Bites:mouse-bite-1mm-3mm, F.Cu at (255.0, 94.3)
- added mouse-bite-1mm-3mm: VAL**, Mouse-Bites:mouse-bite-1mm-3mm, F.Cu at (153.3, 131.0)
- added mouse-bite-1mm-3mm: VAL**, Mouse-Bites:mouse-bite-1mm-3mm, F.Cu at (238.3, 82.4)
- added mouse-bite-1mm-3mm: VAL**, Mouse-Bites:mouse-bite-1mm-3mm, F.Cu at (153.3, 128.0)
- added mouse-bite-1mm-3mm: VAL**, Mouse-Bites:mouse-bite-1mm-3mm, F.Cu at (31.1, 91.3)
- added mouse-bite-1mm-3mm: VAL**, Mouse-Bites:mouse-bite-1mm-3mm, F.Cu at (208.5, 73.8)
- added mouse-bite-1mm-3mm: VAL**, Mouse-Bites:mouse-bite-1mm-3mm, F.Cu at (56.1, 78.9)
- added mouse-bite-1mm-3mm: VAL**, Mouse-Bites:mouse-bite-1mm-3mm, F.Cu at (241.2, 83.6)
- added mouse-bite-1mm-3mm: VAL**, Mouse-Bites:mouse-bite-1mm-3mm, F.Cu at (202.5, 73.8)
- added mouse-bite-1mm-3mm: VAL**, Mouse-Bites:mouse-bite-1mm-3mm, F.Cu at (153.3, 125.0)
- added mouse-bite-1mm-3mm: VAL**, Mouse-Bites:mouse-bite-1mm-3mm, F.Cu at (38.8, 88.5)
- added mouse-bite-1mm-3mm: VAL**, Mouse-Bites:mouse-bite-1mm-3mm, F.Cu at (153.3, 104.0)
- added mouse-bite-1mm-3mm: VAL**, Mouse-Bites:mouse-bite-1mm-3mm, F.Cu at (205.5, 73.8)
- added mouse-bite-1mm-3mm: VAL**, Mouse-Bites:mouse-bite-1mm-3mm, F.Cu at (153.3, 107.0)
- added mouse-bite-1mm-3mm: VAL**, Mouse-Bites:mouse-bite-1mm-3mm, F.Cu at (153.3, 122.0)
- added mouse-bite-1mm-3mm: VAL**, Mouse-Bites:mouse-bite-1mm-3mm, F.Cu at (45.1, 82.2)
- added mouse-bite-1mm-3mm: VAL**, Mouse-Bites:mouse-bite-1mm-3mm, F.Cu at (243.3, 85.7)
- added mouse-bite-1mm-3mm: VAL**, Mouse-Bites:mouse-bite-1mm-3mm, F.Cu at (40.9, 86.4)
- added mouse-bite-1mm-3mm: VAL**, Mouse-Bites:mouse-bite-1mm-3mm, F.Cu at (63.2, 73.5)
- added mouse-bite-1mm-3mm: VAL**, Mouse-Bites:mouse-bite-1mm-3mm, F.Cu at (153.3, 101.0)
- added mouse-bite-1mm-3mm: VAL**, Mouse-Bites:mouse-bite-1mm-3mm, F.Cu at (53.1, 78.9)
- added mouse-bite-1mm-3mm: VAL**, Mouse-Bites:mouse-bite-1mm-3mm, F.Cu at (257.9, 95.5)
- added mouse-bite-1mm-3mm: VAL**, Mouse-Bites:mouse-bite-1mm-3mm, F.Cu at (77.2, 70.2)
- added mouse-bite-1mm-3mm: VAL**, Mouse-Bites:mouse-bite-1mm-3mm, F.Cu at (47.2, 80.1)
- added mouse-bite-1mm-3mm: VAL**, Mouse-Bites:mouse-bite-1mm-3mm, F.Cu at (153.3, 119.0)
- added mouse-bite-1mm-3mm: VAL**, Mouse-Bites:mouse-bite-1mm-3mm, F.Cu at (217.5, 73.8)
- added mouse-bite-1mm-3mm: VAL**, Mouse-Bites:mouse-bite-1mm-3mm, F.Cu at (71.2, 70.2)
- added mouse-bite-1mm-3mm: VAL**, Mouse-Bites:mouse-bite-1mm-3mm, F.Cu at (245.4, 87.8)
- added mouse-bite-1mm-3mm: VAL**, Mouse-Bites:mouse-bite-1mm-3mm, F.Cu at (220.1, 74.9)
- added mouse-bite-1mm-3mm: VAL**, Mouse-Bites:mouse-bite-1mm-3mm, F.Cu at (65.3, 71.4)
- added mouse-bite-1mm-3mm: VAL**, Mouse-Bites:mouse-bite-1mm-3mm, F.Cu at (229.3, 82.4)
- added mouse-bite-1mm-3mm: VAL**, Mouse-Bites:mouse-bite-1mm-3mm, F.Cu at (252.4, 93.2)
- added mouse-bite-1mm-3mm: VAL**, Mouse-Bites:mouse-bite-1mm-3mm, F.Cu at (232.3, 82.4)
- added mouse-bite-1mm-3mm: VAL**, Mouse-Bites:mouse-bite-1mm-3mm, F.Cu at (50.1, 78.9)
- added mouse-bite-1mm-3mm: VAL**, Mouse-Bites:mouse-bite-1mm-3mm, F.Cu at (153.3, 110.0)
- added mouse-bite-1mm-3mm: VAL**, Mouse-Bites:mouse-bite-1mm-3mm, F.Cu at (247.5, 89.9)
- added mouse-bite-1mm-3mm: VAL**, Mouse-Bites:mouse-bite-1mm-3mm, F.Cu at (29.5, 93.3)
- added mouse-bite-1mm-3mm: VAL**, Mouse-Bites:mouse-bite-1mm-3mm, F.Cu at (199.8, 72.5)
- added mouse-bite-1mm-3mm: VAL**, Mouse-Bites:mouse-bite-1mm-3mm, F.Cu at (226.4, 81.2)
- added mouse-bite-1mm-3mm: VAL**, Mouse-Bites:mouse-bite-1mm-3mm, F.Cu at (235.3, 82.4)
- added mouse-bite-1mm-3mm: VAL**, Mouse-Bites:mouse-bite-1mm-3mm, F.Cu at (36.7, 90.6)
- added mouse-bite-1mm-3mm: VAL**, Mouse-Bites:mouse-bite-1mm-3mm, F.Cu at (34.1, 91.3)
- added mouse-bite-1mm-3mm: VAL**, Mouse-Bites:mouse-bite-1mm-3mm, F.Cu at (43.0, 84.3)
- added mouse-bite-1mm-3mm: VAL**, Mouse-Bites:mouse-bite-1mm-3mm, F.Cu at (214.5, 73.8)
- added mouse-bite-1mm-3mm: VAL**, Mouse-Bites:mouse-bite-1mm-3mm, F.Cu at (61.1, 75.6)
- added mouse-bite-1mm-3mm: VAL**, Mouse-Bites:mouse-bite-1mm-3mm, F.Cu at (211.5, 73.8)
- added mouse-bite-1mm-3mm: VAL**, Mouse-Bites:mouse-bite-1mm-3mm, F.Cu at (153.3, 116.0)
- J10, J12, J7, J8: footprint Connector_PinSocket_2.54mm:PinSocket_1x03_P2.54mm_Vertical -> pogo-socket-angled:PinSocket_1x03_P2.54mm_Vertical
- J11, J5, J6, J9: footprint Connector_PinSocket_2.54mm:PinSocket_1x04_P2.54mm_Vertical -> pogo-socket-angled:PinSocket_1x04_P2.54mm_Vertical
- moved J6 295.7 mm to (215.7, 51.6)
- moved D16 294.3 mm to (212.4, 70.0)
- moved D17 294.3 mm to (229.8, 75.3)
- moved D18 294.3 mm to (244.9, 84.3)
- moved D49 294.3 mm to (225.4, 63.3)
- moved D50 294.3 mm to (244.2, 72.2)
- moved D51 294.3 mm to (259.6, 85.0)
- moved SW16 294.3 mm to (221.8, 62.7)
- moved SW17 294.3 mm to (240.8, 70.7)
- moved SW18 294.3 mm to (256.8, 82.7)
- moved J7 292.4 mm to (205.2, 56.9), turned to 0 degrees
- moved J5 227.3 mm to (127.7, 131.8)
- moved R1 226.8 mm to (134.7, 105.2), turned to 0 degrees
- moved D11 225.9 mm to (33.7, 145.2)
- moved J8 225.7 mm to (118.1, 151.7), turned to 180 degrees
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Connections:
- J11 pad 1: /Right Half/Thumbpad/C1 -> /Right Half/Thumbpad/R3
- J11 pad 2: /Right Half/Thumbpad/R1 -> /Right Half/Thumbpad/R2
- J11 pad 3: /Right Half/Thumbpad/R2 -> /Right Half/Thumbpad/R1
- J11 pad 4: /Right Half/Thumbpad/R3 -> /Right Half/Thumbpad/C1
- J12 pad 1: Net-(D67-VDD) -> Net-(D67-VSS)
- J12 pad 3: Net-(D67-VSS) -> Net-(D67-VDD)
- J5 pad 1: /Left Half/R3 -> /Left Half/R2
- J5 pad 2: /Left Half/R2 -> /Left Half/R3
- J6 pad 3: /Left Half/Thumbpad/R2 -> /Left Half/Thumbpad/R3
- J6 pad 4: /Left Half/Thumbpad/R3 -> /Left Half/Thumbpad/R2
- J9 pad 1: /Right Half/R3 -> /Right Half/C6
- J9 pad 2: /Right Half/R2 -> /Right Half/R1
- J9 pad 3: /Right Half/R1 -> /Right Half/R2
- J9 pad 4: /Right Half/C6 -> /Right Half/R3
- R1 pad 1: /Left Half/OUT -> +3V3
- U1 pad 3v3: unconnected-(U1-Pad3v3) -> +3V3
- U1 pad 7: /Left Half/R2 -> /Left Half/R3
- U1 pad 8: /Left Half/R3 -> /Left Half/R2
- U2 pad 14: unconnected-(U2-Pad14) -> /Right Half/R3
- U2 pad 15: /Right Half/C6 -> /Right Half/R2
- U2 pad 26: /Right Half/SDA -> /Right Half/R1
- U2 pad 27: /Right Half/SCL -> /Right Half/C6
- U2 pad 5: /Right Half/R1 -> unconnected-(U2-Pad5)
- U2 pad 6: /Right Half/R2 -> unconnected-(U2-Pad6)
- U2 pad 7: /Right Half/R3 -> unconnected-(U2-Pad7)
Routing:
- net /Left Half/R1: track 264.8 -> 180.9 mm
- net /Right Half/SCL: track 21.9 -> 0.00 mm
- net /Right Half/SDA: track 21.9 -> 0.00 mm
- net GND: track 1014.0 -> 993.6 mm
- net Net-(D52-DOUT): track 91.9 -> 110.7 mm
- net +3V3: track 0.00 -> 18.7 mm
- net /Left Half/ADC0: track 24.2 -> 8.39 mm
- net +5V: track 962.9 -> 978.6 mm
- net /Right Half/R3: track 143.2 -> 128.1 mm
- net Net-(D49-VSS): track 74.2 -> 82.6 mm
- net /Left Half/R3: track 116.4 -> 124.7 mm
- net Net-(D49-VDD): track 66.0 -> 73.6 mm
- net /Right Half/R1: track 158.4 -> 151.1 mm
- net /Right Half/R2: track 126.1 -> 118.9 mm
- net /Left Half/Thumbpad/R3: track 63.9 -> 58.4 mm
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Other:
- board size 4.4 x 4.4 mm -> 266.9 x 104.8 mm
