File: kicad/left_half.kicad_sch (KiCad schematic)
At the start: 52 parts, among them J1 Conn_01x03_Pin, J2 AudioJack4, J5 Conn_01x04_Pin, J8 Conn_01x03_Pin, SW1 SW_Push, SW10 SW_Push, SW11 SW_Push, SW12 SW_Push, SW13 SW_Push, SW14 SW_Push, SW15 SW_Push, SW2 SW_Push, SW3 SW_Push, SW4 SW_Push, SW5 SW_Push, SW6 SW_Push, SW7 SW_Push, SW8 SW_Push, SW9 SW_Push, U1 RP2040-Zero

Commit message: final PCB ready
- bugs: LED position and wiring (wrong by footprint)
Parts:
- removed J1: Conn_01x03_Pin, Connector_PinHeader_2.54mm:PinHeader_1x03_P2.54mm_Vertical, symbol Connector:Conn_01x03_Pin
- J5: footprint Connector_PinSocket_2.54mm:PinSocket_1x04_P2.54mm_Vertical -> pogo-socket-angled:PinSocket_1x04_P2.54mm_Vertical
- J8: footprint Connector_PinSocket_2.54mm:PinSocket_1x03_P2.54mm_Vertical -> pogo-socket-angled:PinSocket_1x03_P2.54mm_Vertical
Connections:
- net OUT is gone; now on net +3V3: R1.1
- net R2: now also J5.1 (Pin_1), U1.8; no longer J5.2 (Pin_2), U1.7
- net R3: now also J5.2 (Pin_2), U1.7; no longer J5.1 (Pin_1), U1.8
- net +3V3: now reaches U1.3v3
Changed lines of the file:
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@@
 		)
 	)
-	(label "GND"
-		(at 214.63 36.83 270)
-		(effects
-			(font
-				(size 1.27 1.27)
-			)
-			(justify right bottom)
-		)
-	)
 	(label "C4"
 		(at 146.05 81.28 0)
@@
 		)
 	)
-	(label "OUT"
-		(at 212.09 36.83 270)
-		(effects
-			(font
-				(size 1.27 1.27)
-			)
-			(justify right bottom)
-		)
-	)
 	(label "C1"
 		(at 88.9 43.18 0)
@@
 		)
 	)
-	(label "OUT"
-		(at 254 31.75 0)
-		(effects
-			(font
-				(size 1.27 1.27)
-			)
-			(justify left bottom)
-		)
-	)
 	(label "ADC0"
 		(at 236.22 83.82 180)
@@
 	)
 	(label "R2"
-		(at 190.5 62.23 180)
+		(at 190.5 64.77 180)
 		(effects
 			(font
@@
 	)
 	(label "R3"
-		(at 190.5 64.77 180)
+		(at 190.5 62.23 180)
 		(effects
 			(font
@@
 	)
 	(label "R2"
-		(at 236.22 106.68 180)
+		(at 236.22 104.14 180)
 		(effects
 			(font
@@
 	)
 	(label "R3"
-		(at 236.22 104.14 180)
+		(at 236.22 106.68 180)
 		(effects
 			(font
@@
 		)
 	)
-	(label "+5V"
-		(at 209.55 36.83 270)
-		(effects
-			(font
-				(size 1.27 1.27)
-			)
-			(justify right bottom)
-		)
-	)
 	(label "GND"
 		(at 228.6 31.75 180)
@@
 			)
 		)
-		(property "Footprint" "Connector_PinSocket_2.54mm:PinSocket_1x03_P2.54mm_Vertical"
+		(property "Footprint" "pogo-socket-angled:PinSocket_1x03_P2.54mm_Vertical"
 			(at 195.58 102.87 0)
 			(effects
@@
 	)
 	(symbol
+		(lib_id "power:+3V3")
+		(at 254 31.75 270)
+		(unit 1)
+		(exclude_from_sim no)
+		(in_bom yes)
+		(on_board yes)
+		(dnp no)
+		(fields_autoplaced yes)
+		(property "Reference" "#PWR03"
+			(at 250.19 31.75 0)
+			(effects
+				(font
+					(size 1.27 1.27)
+				)
+				(hide yes)
+			)
+		)
+		(property "Value" "+3V3"
+			(at 257.81 31.7499 90)
+			(effects
+				(font
+					(size 1.27 1.27)
+				)
+				(justify left)
+			)
+		)
+		(property "Footprint" ""
+			(at 254 31.75 0)
+			(effects
+				(font
+					(size 1.27 1.27)
+				)
+				(hide yes)
+			)
+		)
+		(property "Datasheet" ""
+			(at 254 31.75 0)
+			(effects
+				(font
+					(size 1.27 1.27)
+				)
+				(hide yes)
+			)
+		)
+		(property "Description" "Power symbol creates a global label with name \"+3V3\""
+			(at 254 31.75 0)
+			(effects
+				(font
+					(size 1.27 1.27)
+				)
+				(hide yes)
+			)
+		)
+		(pin "1"
+		)
+		(instances
+			(project ""
+				(path "/de3a30da-dd56-4801-a3f5-765b04aa12e1/effbb08b-3fc5-4b96-83dd-92860f3d7777"
+					(reference "#PWR03")
+					(unit 1)
+				)
+			)
+		)
+	)
+	(symbol
 		(lib_id "Device:D")
 		(at 135.89 46.99 90)
@@
 	)
 	(symbol
+		(lib_id "power:+3V3")
+		(at 236.22 73.66 90)
+		(unit 1)
+		(exclude_from_sim no)
+		(in_bom yes)
+		(on_board yes)
+		(dnp no)
+		(fields_autoplaced yes)
+		(property "Reference" "#PWR06"
+			(at 240.03 73.66 0)
+			(effects
+				(font
+					(size 1.27 1.27)
+				)
+				(hide yes)
+			)
+		)
+		(property "Value" "+3V3"
+			(at 232.41 73.6599 90)
+			(effects
+				(font
+					(size 1.27 1.27)
+				)
+				(justify left)
+			)
+		)
+		(property "Footprint" ""
+			(at 236.22 73.66 0)
+			(effects
+				(font
+					(size 1.27 1.27)
+				)
+				(hide yes)
+			)
+		)
+		(property "Datasheet" ""
+			(at 236.22 73.66 0)
+			(effects
+				(font
+					(size 1.27 1.27)
+				)
+				(hide yes)
+			)
+		)
+		(property "Description" "Power symbol creates a global label with name \"+3V3\""
+			(at 236.22 73.66 0)
+			(effects
+				(font
+					(size 1.27 1.27)
+				)
+				(hide yes)
+			)
+		)
+		(pin "1"
+		)
+		(instances
+			(project ""
+				(path "/de3a30da-dd56-4801-a3f5-765b04aa12e1/effbb08b-3fc5-4b96-83dd-92860f3d7777"
+					(reference "#PWR06")
+					(unit 1)
+				)
+			)
+		)
+	)
+	(symbol
 		(lib_id "Switch:SW_Push")
 		(at 140.97 81.28 0)
@@
 			)
 		)
-		(property "Footprint" "Connector_PinSocket_2.54mm:PinSocket_1x04_P2.54mm_Vertical"
+		(property "Footprint" "pogo-socket-angled:PinSocket_1x04_P2.54mm_Vertical"
 			(at 195.58 62.23 0)
 			(effects
@@
 					(unit 1)
 				)
-			)
-		)
-	)
-	(symbol
-		(lib_id "Connector:Conn_01x03_Pin")
-		(at 212.09 31.75 270)
-		(unit 1)
-		(exclude_from_sim no)
-		(in_bom yes)
-		(on_board yes)
-		(dnp no)
-		(fields_autoplaced yes)
-		(property "Reference" "J1"
-			(at 212.09 26.67 90)
-			(effects
-				(font
-					(size 1.27 1.27)
-				)
-			)
-		)
-		(property "Value" "Conn_01x03_Pin"
-			(at 212.09 29.21 90)
-			(effects
-				(font
-					(size 1.27 1.27)
-				)
-			)
-		)
-		(property "Footprint" "Connector_PinHeader_2.54mm:PinHeader_1x03_P2.54mm_Vertical"
-			(at 212.09 31.75 0)
-			(effects
-				(font
-					(size 1.27 1.27)
-				)
-				(hide yes)
-			)
-		)
-		(property "Datasheet" "~"
-			(at 212.09 31.75 0)
-			(effects
-				(font
-					(size 1.27 1.27)
-				)
-				(hide yes)
-			)
-		)
-		(property "Description" "Placeholder for PIR"
-			(at 212.09 31.75 0)
-			(effects
-				(font
-					(size 1.27 1.27)
-				)
-				(hide yes)
-			)
-		)
-		(pin "1"
-		)
-		(pin "2"
-		)
-		(pin "3"
-		)
-		(instances
-			(project ""
-				(path "/de3a30da-dd56-4801-a3f5-765b04aa12e1/effbb08b-3fc5-4b96-83dd-92860f3d7777"
-					(reference "J1")
-					(unit 1)
-				)
