File: kicad/left_thumbpad.kicad_sch (KiCad schematic)
At the start: 11 parts, among them J6 Conn_01x04_Pin, J7 Conn_01x03_Pin, SW16 SW_Push, SW17 SW_Push, SW18 SW_Push

Commit message: wip: add PCB
- started working on the actual PCB
- however this will be subject to change later
- add footprint for sk6812-mini-e LEDs
Parts:
- D49, D50, D51: footprint LED_SMD:LED_SK6812MINI_PLCC4_3.5x3.5mm_P1.75mm -> SK6812-Mini-E:MX_SK6812MINI-E
- SW16, SW17, SW18: footprint Choc-V1:Kailh-PG1353-Solderable-1U -> Choc-V1:SW_Kailh_Choc_V1
Changed lines of the file:
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@@
 		(instances
 			(project "Keyboard"
-				(path "/de3a30da-dd56-4801-a3f5-765b04aa12e1/d777195d-63e1-45cf-bdcd-083236482c4e/2e4c41b3-22fd-48bd-af7e-ed67fc59d883"
-					(reference "D70")
-					(unit 1)
-				)
 				(path "/de3a30da-dd56-4801-a3f5-765b04aa12e1/effbb08b-3fc5-4b96-83dd-92860f3d7777/b4a3c6d9-ae00-44ee-b05e-f6bf39312733"
 					(reference "D18")
@@
 			)
 		)
-		(property "Footprint" "Choc-V1:Kailh-PG1353-Solderable-1U"
+		(property "Footprint" "Choc-V1:SW_Kailh_Choc_V1"
 			(at 185.42 76.2 0)
 			(effects
@@
 		(instances
 			(project "Keyboard"
-				(path "/de3a30da-dd56-4801-a3f5-765b04aa12e1/d777195d-63e1-45cf-bdcd-083236482c4e/2e4c41b3-22fd-48bd-af7e-ed67fc59d883"
-					(reference "SW34")
-					(unit 1)
-				)
 				(path "/de3a30da-dd56-4801-a3f5-765b04aa12e1/effbb08b-3fc5-4b96-83dd-92860f3d7777/b4a3c6d9-ae00-44ee-b05e-f6bf39312733"
 					(reference "SW16")
@@
 			)
 		)
-		(property "Footprint" "LED_SMD:LED_SK6812MINI_PLCC4_3.5x3.5mm_P1.75mm"
+		(property "Footprint" "SK6812-Mini-E:MX_SK6812MINI-E"
 			(at 176.53 153.67 0)
 			(effects
@@
 		(instances
 			(project "Keyboard"
-				(path "/de3a30da-dd56-4801-a3f5-765b04aa12e1/d777195d-63e1-45cf-bdcd-083236482c4e/2e4c41b3-22fd-48bd-af7e-ed67fc59d883"
-					(reference "D67")
-					(unit 1)
-				)
 				(path "/de3a30da-dd56-4801-a3f5-765b04aa12e1/effbb08b-3fc5-4b96-83dd-92860f3d7777/b4a3c6d9-ae00-44ee-b05e-f6bf39312733"
 					(reference "D49")
@@
 			)
 		)
-		(property "Footprint" "Choc-V1:Kailh-PG1353-Solderable-1U"
+		(property "Footprint" "Choc-V1:SW_Kailh_Choc_V1"
 			(at 185.42 114.3 0)
 			(effects
@@
 		(instances
 			(project "Keyboard"
-				(path "/de3a30da-dd56-4801-a3f5-765b04aa12e1/d777195d-63e1-45cf-bdcd-083236482c4e/2e4c41b3-22fd-48bd-af7e-ed67fc59d883"
-					(reference "SW36")
-					(unit 1)
-				)
 				(path "/de3a30da-dd56-4801-a3f5-765b04aa12e1/effbb08b-3fc5-4b96-83dd-92860f3d7777/b4a3c6d9-ae00-44ee-b05e-f6bf39312733"
 					(reference "SW18")
@@
 		(instances
 			(project "Keyboard"
-				(path "/de3a30da-dd56-4801-a3f5-765b04aa12e1/d777195d-63e1-45cf-bdcd-083236482c4e/2e4c41b3-22fd-48bd-af7e-ed67fc59d883"
-					(reference "J12")
-					(unit 1)
-				)
 				(path "/de3a30da-dd56-4801-a3f5-765b04aa12e1/effbb08b-3fc5-4b96-83dd-92860f3d7777/b4a3c6d9-ae00-44ee-b05e-f6bf39312733"
 					(reference "J7")
@@
 			)
 		)
-		(property "Footprint" "Choc-V1:Kailh-PG1353-Solderable-1U"
+		(property "Footprint" "Choc-V1:SW_Kailh_Choc_V1"
 			(at 185.42 95.25 0)
 			(effects
@@
 		(instances
 			(project "Keyboard"
-				(path "/de3a30da-dd56-4801-a3f5-765b04aa12e1/d777195d-63e1-45cf-bdcd-083236482c4e/2e4c41b3-22fd-48bd-af7e-ed67fc59d883"
-					(reference "SW35")
-					(unit 1)
-				)
 				(path "/de3a30da-dd56-4801-a3f5-765b04aa12e1/effbb08b-3fc5-4b96-83dd-92860f3d7777/b4a3c6d9-ae00-44ee-b05e-f6bf39312733"
 					(reference "SW17")
@@
 		(instances
 			(project "Keyboard"
-				(path "/de3a30da-dd56-4801-a3f5-765b04aa12e1/d777195d-63e1-45cf-bdcd-083236482c4e/2e4c41b3-22fd-48bd-af7e-ed67fc59d883"
-					(reference "D69")
-					(unit 1)
-				)
 				(path "/de3a30da-dd56-4801-a3f5-765b04aa12e1/effbb08b-3fc5-4b96-83dd-92860f3d7777/b4a3c6d9-ae00-44ee-b05e-f6bf39312733"
 					(reference "D17")
@@
 			)
 		)
-		(property "Footprint" "LED_SMD:LED_SK6812MINI_PLCC4_3.5x3.5mm_P1.75mm"
+		(property "Footprint" "SK6812-Mini-E:MX_SK6812MINI-E"
 			(at 200.66 153.67 0)
 			(effects
@@
 		(instances
 			(project "Keyboard"
-				(path "/de3a30da-dd56-4801-a3f5-765b04aa12e1/d777195d-63e1-45cf-bdcd-083236482c4e/2e4c41b3-22fd-48bd-af7e-ed67fc59d883"
-					(reference "D71")
-					(unit 1)
-				)
 				(path "/de3a30da-dd56-4801-a3f5-765b04aa12e1/effbb08b-3fc5-4b96-83dd-92860f3d7777/b4a3c6d9-ae00-44ee-b05e-f6bf39312733"
 					(reference "D50")
@@
 		(instances
 			(project "Keyboard"
-				(path "/de3a30da-dd56-4801-a3f5-765b04aa12e1/d777195d-63e1-45cf-bdcd-083236482c4e/2e4c41b3-22fd-48bd-af7e-ed67fc59d883"
-					(reference "D68")
-					(unit 1)
-				)
 				(path "/de3a30da-dd56-4801-a3f5-765b04aa12e1/effbb08b-3fc5-4b96-83dd-92860f3d7777/b4a3c6d9-ae00-44ee-b05e-f6bf39312733"
 					(reference "D16")
@@
 			)
 		)
-		(property "Footprint" "LED_SMD:LED_SK6812MINI_PLCC4_3.5x3.5mm_P1.75mm"
+		(property "Footprint" "SK6812-Mini-E:MX_SK6812MINI-E"
 			(at 224.79 153.67 0)
 			(effects
@@
 		(instances
 			(project "Keyboard"
-				(path "/de3a30da-dd56-4801-a3f5-765b04aa12e1/d777195d-63e1-45cf-bdcd-083236482c4e/2e4c41b3-22fd-48bd-af7e-ed67fc59d883"
-					(reference "D72")
-					(unit 1)
-				)
 				(path "/de3a30da-dd56-4801-a3f5-765b04aa12e1/effbb08b-3fc5-4b96-83dd-92860f3d7777/b4a3c6d9-ae00-44ee-b05e-f6bf39312733"
 					(reference "D51")
@@
 		(instances
 			(project "Keyboard"
-				(path "/de3a30da-dd56-4801-a3f5-765b04aa12e1/d777195d-63e1-45cf-bdcd-083236482c4e/2e4c41b3-22fd-48bd-af7e-ed67fc59d883"
-					(reference "J11")
-					(unit 1)
-				)
 				(path "/de3a30da-dd56-4801-a3f5-765b04aa12e1/effbb08b-3fc5-4b96-83dd-92860f3d7777/b4a3c6d9-ae00-44ee-b05e-f6bf39312733"
 					(reference "J6")

Commit message: wip: pcb for both halves
Parts:
- SW16, SW17, SW18: footprint Choc-V1:SW_Kailh_Choc_V1 -> Choc-V1:SW_Kailh_Choc_V1_THT
Connections:
- new net C1: J6.1 (Pin_1), SW16.2, SW17.2, SW18.2
- new net R1: D16.1 (K), J6.2 (Pin_2)
- new net R2: D17.1 (K), J6.3 (Pin_3)
- new net R3: D18.1 (K), J6.4 (Pin_4)

Commit message: final PCB ready
- bugs: LED position and wiring (wrong by footprint)
Parts:
- J6: footprint Connector_PinSocket_2.54mm:PinSocket_1x04_P2.54mm_Vertical -> pogo-socket-angled:PinSocket_1x04_P2.54mm_Vertical
- J7: footprint Connector_PinSocket_2.54mm:PinSocket_1x03_P2.54mm_Vertical -> pogo-socket-angled:PinSocket_1x03_P2.54mm_Vertical
Connections:
- net R2: now also J6.4 (Pin_4); no longer J6.3 (Pin_3)
- net R3: now also J6.3 (Pin_3); no longer J6.4 (Pin_4)
Changed lines of the file:
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@@
+	(wire
+		(pts
+			(xy 140.97 148.59) (xy 157.48 148.59)
+		)
+		(stroke
+			(width 0)
+			(type default)
+		)
+	)
 	(wire
 		(pts
@@
 	(wire
 		(pts
-			(xy 140.97 146.05) (xy 167.64 146.05)
+			(xy 140.97 143.51) (xy 157.48 143.51)
 		)
 		(stroke
@@
 	(wire
 		(pts
-			(xy 175.26 138.43) (xy 199.39 138.43)
+			(xy 140.97 146.05) (xy 167.64 146.05)
 		)
 		(stroke
@@
 	(wire
 		(pts
-			(xy 207.01 146.05) (xy 215.9 146.05)
+			(xy 175.26 138.43) (xy 199.39 138.43)
 		)
 		(stroke
@@
 	(wire
 		(pts
-			(xy 140.97 148.59) (xy 157.48 148.59)
+			(xy 207.01 146.05) (xy 215.9 146.05)
 		)
 		(stroke
@@
 		)
 	)
-	(wire
-		(pts
-			(xy 140.97 143.51) (xy 157.48 143.51)
-		)
-		(stroke
-			(width 0)
-			(type default)
-		)
-	)
 	(label "R2"
-		(at 140.97 104.14 0)
+		(at 140.97 106.68 0)
 		(effects
 			(font
@@
 	)
 	(label "R3"
-		(at 140.97 106.68 0)
+		(at 140.97 104.14 0)
 		(effects
 			(font
@@
 			)
 		)
-		(property "Footprint" "Connector_PinSocket_2.54mm:PinSocket_1x03_P2.54mm_Vertical"
+		(property "Footprint" "pogo-socket-angled:PinSocket_1x03_P2.54mm_Vertical"
 			(at 135.89 146.05 0)
 			(effects
@@
 			)
 		)
-		(property "Footprint" "Connector_PinSocket_2.54mm:PinSocket_1x04_P2.54mm_Vertical"
+		(property "Footprint" "pogo-socket-angled:PinSocket_1x04_P2.54mm_Vertical"
 			(at 135.89 101.6 0)
 			(effects
