File: kicad/right_thumbpad.kicad_sch (KiCad schematic)
At the start: 11 parts, among them J11 Conn_01x04_Pin, J12 Conn_01x03_Pin, SW34 SW_Push, SW35 SW_Push, SW36 SW_Push

Commit message: wip: add PCB
- started working on the actual PCB
- however this will be subject to change later
- add footprint for sk6812-mini-e LEDs
Parts:
- D67, D71, D72: footprint LED_SMD:LED_SK6812MINI_PLCC4_3.5x3.5mm_P1.75mm -> SK6812-Mini-E:MX_SK6812MINI-E
- SW34, SW35, SW36: footprint Choc-V1:Kailh-PG1353-Solderable-1U -> Choc-V1:SW_Kailh_Choc_V1
Changed lines of the file:
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@@
-					(unit 1)
-				)
-				(path "/de3a30da-dd56-4801-a3f5-765b04aa12e1/effbb08b-3fc5-4b96-83dd-92860f3d7777/b4a3c6d9-ae00-44ee-b05e-f6bf39312733"
-					(reference "D18")
 					(unit 1)
 				)
@@
 			)
 		)
-		(property "Footprint" "Choc-V1:Kailh-PG1353-Solderable-1U"
+		(property "Footprint" "Choc-V1:SW_Kailh_Choc_V1"
 			(at 185.42 76.2 0)
 			(effects
@@
 					(unit 1)
 				)
-				(path "/de3a30da-dd56-4801-a3f5-765b04aa12e1/effbb08b-3fc5-4b96-83dd-92860f3d7777/b4a3c6d9-ae00-44ee-b05e-f6bf39312733"
-					(reference "SW16")
-					(unit 1)
-				)
 			)
 		)
@@
 			)
 		)
-		(property "Footprint" "LED_SMD:LED_SK6812MINI_PLCC4_3.5x3.5mm_P1.75mm"
+		(property "Footprint" "SK6812-Mini-E:MX_SK6812MINI-E"
 			(at 176.53 153.67 0)
 			(effects
@@
 					(unit 1)
 				)
-				(path "/de3a30da-dd56-4801-a3f5-765b04aa12e1/effbb08b-3fc5-4b96-83dd-92860f3d7777/b4a3c6d9-ae00-44ee-b05e-f6bf39312733"
-					(reference "D49")
-					(unit 1)
-				)
 			)
 		)
@@
 			)
 		)
-		(property "Footprint" "Choc-V1:Kailh-PG1353-Solderable-1U"
+		(property "Footprint" "Choc-V1:SW_Kailh_Choc_V1"
 			(at 185.42 114.3 0)
 			(effects
@@
 					(unit 1)
 				)
-				(path "/de3a30da-dd56-4801-a3f5-765b04aa12e1/effbb08b-3fc5-4b96-83dd-92860f3d7777/b4a3c6d9-ae00-44ee-b05e-f6bf39312733"
-					(reference "SW18")
-					(unit 1)
-				)
 			)
 		)
@@
 					(unit 1)
 				)
-				(path "/de3a30da-dd56-4801-a3f5-765b04aa12e1/effbb08b-3fc5-4b96-83dd-92860f3d7777/b4a3c6d9-ae00-44ee-b05e-f6bf39312733"
-					(reference "J7")
-					(unit 1)
-				)
 			)
 		)
@@
 			)
 		)
-		(property "Footprint" "Choc-V1:Kailh-PG1353-Solderable-1U"
+		(property "Footprint" "Choc-V1:SW_Kailh_Choc_V1"
 			(at 185.42 95.25 0)
 			(effects
@@
 					(unit 1)
 				)
-				(path "/de3a30da-dd56-4801-a3f5-765b04aa12e1/effbb08b-3fc5-4b96-83dd-92860f3d7777/b4a3c6d9-ae00-44ee-b05e-f6bf39312733"
-					(reference "SW17")
-					(unit 1)
-				)
 			)
 		)
@@
 					(unit 1)
 				)
-				(path "/de3a30da-dd56-4801-a3f5-765b04aa12e1/effbb08b-3fc5-4b96-83dd-92860f3d7777/b4a3c6d9-ae00-44ee-b05e-f6bf39312733"
-					(reference "D17")
-					(unit 1)
-				)
 			)
 		)
@@
 			)
 		)
-		(property "Footprint" "LED_SMD:LED_SK6812MINI_PLCC4_3.5x3.5mm_P1.75mm"
+		(property "Footprint" "SK6812-Mini-E:MX_SK6812MINI-E"
 			(at 200.66 153.67 0)
 			(effects
@@
 					(unit 1)
 				)
-				(path "/de3a30da-dd56-4801-a3f5-765b04aa12e1/effbb08b-3fc5-4b96-83dd-92860f3d7777/b4a3c6d9-ae00-44ee-b05e-f6bf39312733"
-					(reference "D50")
-					(unit 1)
-				)
 			)
 		)
@@
 					(unit 1)
 				)
-				(path "/de3a30da-dd56-4801-a3f5-765b04aa12e1/effbb08b-3fc5-4b96-83dd-92860f3d7777/b4a3c6d9-ae00-44ee-b05e-f6bf39312733"
-					(reference "D16")
-					(unit 1)
-				)
 			)
 		)
@@
 			)
 		)
-		(property "Footprint" "LED_SMD:LED_SK6812MINI_PLCC4_3.5x3.5mm_P1.75mm"
+		(property "Footprint" "SK6812-Mini-E:MX_SK6812MINI-E"
 			(at 224.79 153.67 0)
 			(effects
@@
 					(unit 1)
 				)
-				(path "/de3a30da-dd56-4801-a3f5-765b04aa12e1/effbb08b-3fc5-4b96-83dd-92860f3d7777/b4a3c6d9-ae00-44ee-b05e-f6bf39312733"
-					(reference "D51")
-					(unit 1)
-				)
 			)
 		)
@@
 					(unit 1)
 				)
-				(path "/de3a30da-dd56-4801-a3f5-765b04aa12e1/effbb08b-3fc5-4b96-83dd-92860f3d7777/b4a3c6d9-ae00-44ee-b05e-f6bf39312733"
-					(reference "J6")
-					(unit 1)
-				)

Commit message: wip: pcb for both halves
Parts:
- SW34, SW35, SW36: footprint Choc-V1:SW_Kailh_Choc_V1 -> Choc-V1:SW_Kailh_Choc_V1_THT
Connections:
- new net C1: J11.1 (Pin_1), SW34.2, SW35.2, SW36.2
- new net R1: D68.1 (K), J11.2 (Pin_2)
- new net R2: D69.1 (K), J11.3 (Pin_3)
- new net R3: D70.1 (K), J11.4 (Pin_4)

Commit message: final PCB ready
- bugs: LED position and wiring (wrong by footprint)
Parts:
- J11: footprint Connector_PinSocket_2.54mm:PinSocket_1x04_P2.54mm_Vertical -> pogo-socket-angled:PinSocket_1x04_P2.54mm_Vertical
- J12: footprint Connector_PinSocket_2.54mm:PinSocket_1x03_P2.54mm_Vertical -> pogo-socket-angled:PinSocket_1x03_P2.54mm_Vertical
Connections:
- net C1: now also J11.4 (Pin_4); no longer J11.1 (Pin_1)
- net R1: now also J11.3 (Pin_3); no longer J11.2 (Pin_2)
- net R2: now also J11.2 (Pin_2); no longer J11.3 (Pin_3)
- net R3: now also J11.1 (Pin_1); no longer J11.4 (Pin_4)
- net at D67.2 (VSS), D71.2 (VSS), D72.2 (VSS): now also J12.1 (Pin_1); no longer J12.3 (Pin_3)
- net at D67.4 (VDD), D71.4 (VDD), D72.4 (VDD): now also J12.3 (Pin_3); no longer J12.1 (Pin_1)
Other:
- moved on the sheet: J11
Changed lines of the file:
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@@
+	(wire
+		(pts
+			(xy 140.97 143.51) (xy 157.48 143.51)
+		)
+		(stroke
+			(width 0)
+			(type default)
+		)
+	)
+	(wire
+		(pts
+			(xy 157.48 153.67) (xy 175.26 153.67)
+		)
+		(stroke
+			(width 0)
+			(type default)
+		)
+	)
+	(wire
+		(pts
+			(xy 182.88 146.05) (xy 191.77 146.05)
+		)
+		(stroke
+			(width 0)
+			(type default)
+		)
+	)
 	(wire
 		(pts
@@
 		)
 	)
-	(wire
-		(pts
-			(xy 157.48 153.67) (xy 175.26 153.67)
-		)
-		(stroke
-			(width 0)
-			(type default)
-		)
-	)
-	(wire
-		(pts
-			(xy 182.88 146.05) (xy 191.77 146.05)
-		)
-		(stroke
-			(width 0)
-			(type default)
-		)
-	)
-	(wire
-		(pts
-			(xy 140.97 143.51) (xy 157.48 143.51)
-		)
-		(stroke
-			(width 0)
-			(type default)
-		)
-	)
 	(label "C1"
-		(at 140.97 99.06 0)
+		(at 140.97 96.52 0)
 		(effects
 			(font
@@
 	)
 	(label "R2"
-		(at 140.97 104.14 0)
+		(at 140.97 101.6 0)
 		(effects
 			(font
@@
 	)
 	(label "R3"
-		(at 140.97 106.68 0)
+		(at 140.97 104.14 0)
 		(effects
 			(font
@@
 	)
 	(label "R1"
-		(at 140.97 101.6 0)
+		(at 140.97 99.06 0)
 		(effects
 			(font
@@
 		(lib_id "Connector:Conn_01x03_Pin")
 		(at 135.89 146.05 0)
+		(mirror x)
 		(unit 1)
 		(exclude_from_sim no)
@@
 		(fields_autoplaced yes)
 		(property "Reference" "J12"
-			(at 136.525 138.43 0)
+			(at 136.525 153.67 0)
 			(effects
 				(font
@@
 		)
 		(property "Value" "Conn_01x03_Pin"
-			(at 136.525 140.97 0)
-			(effects
-				(font
-					(size 1.27 1.27)
-				)
-			)
-		)
-		(property "Footprint" "Connector_PinSocket_2.54mm:PinSocket_1x03_P2.54mm_Vertical"
+			(at 136.525 151.13 0)
+			(effects
+				(font
+					(size 1.27 1.27)
+				)
+			)
+		)
+		(property "Footprint" "pogo-socket-angled:PinSocket_1x03_P2.54mm_Vertical"
 			(at 135.89 146.05 0)
 			(effects
@@
 		(lib_id "Connector:Conn_01x04_Pin")
 		(at 135.89 101.6 0)
+		(mirror x)
 		(unit 1)
 		(exclude_from_sim no)
@@
 		(fields_autoplaced yes)
 		(property "Reference" "J11"
-			(at 136.525 93.98 0)
+			(at 136.525 109.22 0)
 			(effects
 				(font
@@
 		)
 		(property "Value" "Conn_01x04_Pin"
-			(at 136.525 96.52 0)
-			(effects
-				(font
-					(size 1.27 1.27)
-				)
-			)
-		)
-		(property "Footprint" "Connector_PinSocket_2.54mm:PinSocket_1x04_P2.54mm_Vertical"
+			(at 136.525 106.68 0)
+			(effects
+				(font
+					(size 1.27 1.27)
+				)
+			)
+		)
+		(property "Footprint" "pogo-socket-angled:PinSocket_1x04_P2.54mm_Vertical"
 			(at 135.89 101.6 0)
 			(effects
